Commit message: slam added

File: description/gebot_core.xacro (robot description, xacro)
@@ -45,4 +45,12 @@
     <!-- Robot Base -->
     <link name="base_link"/>
+    <!-- Base_footprint -->
+    <!-- <link name="base_footprint_joint"/>
+    <joint name="base_footprint_joint" type="fixed">
+        <parent link="base_link"/>
+        <child link="base_footprint"/>
+        <origin xyz="0 0 0" rpy="0 0 0"/>
+    </joint> -->
+    <!-- Chassis -->
     <link name="base_chassis">
         <collision>

File: description/robot.urdf.xacro (robot description, xacro)
@@ -9,5 +9,5 @@
     <!-- <xacro:include filename="gazebo_control.xacro" /> -->
     <!-- <xacro:include filename="ros2_control.xacro" /> -->
-    <!-- <xacro:include filename="tricycle_control.xacro" /> -->
+    <xacro:include filename="tricycle_control.xacro" />
     <!-- <xacro:include filename="tricycle_steering_control.xacro" /> -->
 </robot>

File: description/tricycle_steering_control.xacro (robot description, xacro)
@@ -5,5 +5,5 @@
             <plugin>gazebo_ros2_control/GazeboSystem</plugin>
         </hardware>
-        <joint name="front_steering_joint">
+        <joint name="front_wheel_joint">
             <command_interface name="position"/>
             <state_interface name="position" />
