Commit message: Modified the model

File: description/body.xacro (robot description, xacro)
@@ -5,5 +5,5 @@
         <visual>
             <geometry>
-                <box size="0.9 0.9 0.3"/>
+                <box size="0.9 0.9 0.55"/>
             </geometry>
             <material name="myblue"/>
@@ -11,13 +11,55 @@
         <collision>
             <geometry>
-                <box size="0.9 0.9 0.3"/>
+                <box size="0.9 0.9 0.55"/>
             </geometry>
         </collision>
-        <xacro:box_inertia m="1" w="0.8" d="0.9" h="0.3"/><!--10-->
+        <xacro:box_inertia m="1" w="0.9" d="0.9" h="0.55"/><!--10-->
+    </link>
+    <link name="control_box">
+        <visual>
+            <geometry>
+                <box size="0.2 0.4 0.35"/>
+            </geometry>
+            <material name="white"/>
+        </visual>
+        <collision>
+            <geometry>
+                <box size="0.2 0.4 0.35"/>
+            </geometry>
+        </collision>
+        <xacro:box_inertia m="1" w="0.2" d="0.4" h="0.35"/>
+    </link>
+    <link name="seat">
+        <visual>
+            <geometry>
+                <box size="0.4 0.38 0.1"/>
+            </geometry>
+            <material name="black"/>
+        </visual>
+        <collision>
+            <geometry>
+                <box size="0.4 0.38 0.075"/>
+            </geometry>
+        </collision>
+        <xacro:box_inertia m="1" w="0.4" d="0.38" h="0.075"/>
+    </link>
+    <link name="seatback">
+        <visual>
+            <geometry>
+                <box size="0.1 0.38 0.45"/>
+            </geometry>
+            <material name="black"/>
+        </visual>
+        <collision>
+            <geometry>
+                <box size="0.1 0.38 0.45"/>
+            </geometry>
+        </collision>
+        <xacro:box_inertia m="1" w="0.1" d="0.38" h="0.45"/>
     </link>
     <link name="chassis2">
         <visual>
             <geometry>
-                <box size="0.5 0.9 0.35"/>
+                <box size="0.075 0.4 0.6"/>
             </geometry>
             <material name="myblue"/>
@@ -25,39 +67,35 @@
         <collision>
             <geometry>
-                <box size="0.5 0.9 0.35"/>
+                <box size="0.075 0.4 0.6"/>
             </geometry>
         </collision>
-        <xacro:box_inertia m="1" w="0.5" d="0.9" h="0.35"/><!--3-->
-    </link>
-    <link name="chassis3">
-        <visual>
-            <geometry>
-                <box size="0.15 0.6 0.2"/>
-            </geometry>
-            <material name="myblue"/>
-        </visual>
-        <collision>
-            <geometry>
-                <box size="0.15 0.6 0.2"/>
-            </geometry>
-        </collision>
-        <xacro:box_inertia m="1" w="0.6" d="0.15" h="0.2"/>
+        <xacro:box_inertia m="1" w="0.075" d="0.4" h="0.6"/><!--10-->
     </link>
     <joint name="base_to_chassis1" type="fixed">
         <parent link="base_chassis"/>
         <child link="chassis1"/>
-        <origin xyz="-0.25 0.0 0.225"/>
+        <origin xyz="-0.225 0.0 0.3"/>
     </joint>
-    <joint name="chassis1_to_chassis2" type="fixed">
+    <joint name="chassis1_to_control_box" type="fixed">
         <!--axis xyz="0 1 0"/-->
         <!--limit effort="1000.0" lower="-0.4" upper="0.4" velocity="0.5"/-->
         <parent link="chassis1"/>
+        <child link="control_box"/>
+        <origin xyz="-0.05 0.0 0.45"/>
+    </joint>
+    <joint name="base_to_seat" type="fixed">
+        <parent link="chassis1"/>
+        <child link="seat"/>
+        <origin xyz="0.25 0.0 0.275"/>
+    </joint>
+    <joint name="seat_to_seatback" type="fixed">
+        <parent link="seat"/>
+        <child link="seatback"/>
+        <origin xyz="-0.15 0.0 0.0"/>
+    </joint>
+    <joint name="base_to_chassis2" type="fixed">
+        <parent link="base_chassis"/>
         <child link="chassis2"/>
-        <origin xyz="-0.2 0.0 0.325"/>
-    </joint>
-    <joint name="base_to_chassis3" type="fixed">
-        <parent link="base_chassis"/>
-        <child link="chassis3"/>
-        <origin xyz="0.6 0.0 0.125"/>
+        <origin xyz="0.6385 0.0 0.325"/>
     </joint>
 </robot>

File: description/gazebo_control.xacro (robot description, xacro)
@@ -9,5 +9,5 @@
             <right_joint>right_wheel_joint</right_joint>
             <wheel_separation>0.9</wheel_separation>
-            <wheel_diameter>0.2</wheel_diameter>
+            <wheel_diameter>0.25</wheel_diameter>
             <!-- Limits -->
             <max_wheel_torque>200</max_wheel_torque>

File: description/gazebo_material.xacro (robot description, xacro)
@@ -1,7 +1,4 @@
 <?xml version="1.0"?>
-<robot xmlns:xacro="http://www.ros.org/wiki/xacro">
-    <gazebo reference="base_chassis">
-        <material>Gazebo/White</material>
-    </gazebo>
+<robot xmlns:xacro="http://www.ros.org/wiki/xacro" name="gebot">
     <gazebo reference="base_chassis">
         <material>Gazebo/White</material>
@@ -27,5 +24,11 @@
         <material>Gazebo/White</material>
     </gazebo>
-    <gazebo reference="connection">
+    <gazebo reference="chain_frame">
+        <material>Gazebo/Yellow</material>
+    </gazebo>
+    <gazebo reference="bearing">
+        <material>Gazebo/Black</material>
+    </gazebo>
+    <gazebo reference="bearing_gear">
         <material>Gazebo/Yellow</material>
     </gazebo>
@@ -40,6 +43,12 @@
         <material>Gazebo/SkyBlue</material>
     </gazebo>
-    <gazebo reference="chassis3">
-        <material>Gazebo/SkyBlue</material>
+    <gazebo reference="control_box">
+        <material>Gazebo/White</material>
+    </gazebo>
+    <gazebo reference="seat">
+        <material>Gazebo/Grey</material>
+    </gazebo>
+    <gazebo reference="seatback">
+        <material>Gazebo/Grey</material>
     </gazebo>
     <!-- Lidar -->
@@ -47,3 +56,7 @@
         <material>Gazebo/Red</material>
     </gazebo>
+    <!-- Camera -->
+    <gazebo reference="camera_frame">
+        <material>Gazebo/Red</material>
+    </gazebo>
 </robot>

File: description/gebot_urdf.xacro (robot description, xacro)
@@ -46,10 +46,10 @@
     <link name="base_link"/>
     <!-- Base_footprint -->
-    <!-- <link name="base_footprint_joint"/>
+    <!--<link name="base_footprint_joint"/>
     <joint name="base_footprint_joint" type="fixed">
         <parent link="base_link"/>
         <child link="base_footprint"/>
         <origin xyz="0 0 0" rpy="0 0 0"/>
-    </joint> -->
+    </joint>-->
     <!-- Chassis -->
     <link name="base_chassis">
@@ -67,5 +67,5 @@
             <material name="base"/>
         </visual>
-        <xacro:box_inertia m="3" w="${base_width}" d="${base_length}" h="${base_height}"/>
+        <xacro:box_inertia m="1" w="${base_width}" d="${base_length}" h="${base_height}"/><!--3-->
     </link>
     <joint name="base_link_joint" type="fixed">
@@ -117,11 +117,12 @@
             </geometry>
         </collision>
-        <xacro:cylinder_inertia m="5" r="${wheel_radius}" h="${(wheel_width+0.02)}"/>
+        <xacro:cylinder_inertia m="1" r="${wheel_radius}" h="${(wheel_width+0.02)}"/><!--5-->
     </link>
     <!--<joint name="front_wheel_joint" type="continuous">
-        <axis xyz="0 1 0"/>
-        <parent link="base_link"/>
+        <axis xyz="0 0 1"/>
+        <parent link="base_chassis"/>
         <child link="front_wheel"/>
-        <origin xyz="0.5 0.0 -0.125"/>
+        <origin xyz="0.475 0.0 -0.145" rpy="${-pi/2} 0 0"/>
+        <dynamics damping="0.2" />
     </joint>-->
     <!-- Steering Links and Joints-->
@@ -140,14 +141,19 @@
             </geometry>
         </collision>
-        <xacro:cylinder_inertia m="0.01" r="0.02" h="0.93"/>
-    </link>
-    <joint name="front_steering_joint" type="revolute">
+        <xacro:cylinder_inertia m="1" r="0.02" h="0.93"/><!--0.01-->
+    </link>
+    <!--<joint name="front_steering_joint" type="revolute">
         <axis xyz="0 0 1"/>
         <limit effort="1000.0" lower="-1.4" upper="1.4" velocity="0.5"/>
         <parent link="base_chassis"/>
         <child link="steering_link"/>
-        <origin xyz="0.66 0.0 0.4"/>
-    </joint>
-    <link name="chain_frame">
+        <origin xyz="0.65 0.0 0.4"/>
+    </joint>-->
+    <joint name="front_steering_joint" type="fixed">
+        <parent link="base_chassis"/>
+        <child link="steering_link"/>
+        <origin xyz="0.65 0.0 0.4"/>
+    </joint>
+    <!--<link name="chain_frame">
         <visual>
             <origin xyz="0.0 0.0 0.0" rpy="0.0 ${pi/2} 0.0"/>
@@ -169,41 +175,20 @@
         <child link="chain_frame"/>
         <origin xyz="-0.1 0.0 -0.465"/>
-    </joint>
-    <!--link name="connection">
+    </joint>-->
+    <link name="steering_wheel">
         <visual>
             <origin xyz="0.0 0.0 0.0" rpy="${pi/2} 0.0 0.0"/>
             <geometry>
-                <cylinder radius="0.01" length="0.05"/>
-            </geometry>
-            <material name="myblue"/>
+                <cylinder radius="0.02" length="0.3"/>
+            </geometry>
+            <material name="black"/>
         </visual>
         <collision>
             <origin xyz="0.0 0.0 0.0" rpy="${pi/2} 0.0 0.0"/>
             <geometry>
-                <cylinder radius="0.01" length="0.05"/>
-            </geometry>
-        </collision>
-        <xacro:cylinder_inertia m="0.001" r="0.01" h="0.05"/>
-    </link>
-    <joint name="steering_connector"  type="fixed">
-        <parent link="chain_frame"/>
-        <child link="connection"/>
-        <origin xyz="-0.2 0.0 0.0"/>
-    </joint-->
-    <link name="steering_wheel">
-        <visual>
-            <origin xyz="0.0 0.0 0.0" rpy="${pi/2} 0.0 0.0"/>
-            <geometry>
                 <cylinder radius="0.02" length="0.3"/>
             </geometry>
-            <material name="black"/>
-        </visual>
-        <collision>
-            <origin xyz="0.0 0.0 0.0" rpy="${pi/2} 0.0 0.0"/>
-            <geometry>
-                <cylinder radius="0.02" length="0.3"/>
-            </geometry>
-        </collision>
-        <xacro:cylinder_inertia m="0.005" r="0.02" h="0.3"/>
+        </collision>
+        <xacro:cylinder_inertia m="1" r="0.02" h="0.3"/><!--0.005-->
     </link>
     <joint name="steering_wheel_connector" type="fixed">
@@ -212,5 +197,58 @@
         <origin xyz="0.0 0.0 0.465"/>
     </joint>
+    <link name="bearing">
+        <visual>
+            <origin xyz="0.0 0.0 0.0" rpy="0.0 0.0 0.0"/>
+            <geometry>
+                <cylinder radius="0.045" length="0.04"/><!--0.04-->
+            </geometry>
+            <material name="myblue"/>
+        </visual>
+        <collision>
+            <origin xyz="0.0 0.0 0.0" rpy="0.0 0.0 0.0"/>
+            <geometry>
+                <cylinder radius="0.045" length="0.04"/>
+            </geometry>
+        </collision>
+        <xacro:cylinder_inertia m="1" r="0.0045" h="0.04"/><!--0.001-->
+    </link>
+    <joint name="bearing_joint"  type="revolute">
+        <axis xyz="0 0 1"/>
+        <limit effort="1000.0" lower="-1.4" upper="1.4" velocity="0.5"/>
+        <parent link="base_chassis"/>
+        <child link="bearing"/>
+        <origin xyz="0.475 0.0 0.045"/><!--0.045-->
+    </joint>
+    <link name="bearing_gear">
+        <visual>
+            <origin xyz="0.0 0.0 0.0" rpy="0.0 0.0 0.0"/>
+            <geometry>
+                <cylinder radius="0.02" length="0.195"/>
+            </geometry>
+            <material name="myblue"/>
+        </visual>
+        <collision>
+            <origin xyz="0.0 0.0 0.0" rpy="0.0 0.0 0.0"/>
+            <geometry>
+                <cylinder radius="0.02" length="0.195"/>
+            </geometry>
+        </collision>
+        <xacro:cylinder_inertia m="1" r="0.02" h="0.195"/><!--0.001-->
+    </link>
+    <joint name="drive_unit" type="fixed">
+        <parent link="bearing"/>
+        <child link="bearing_gear"/>
+        <origin xyz="0.0 0.0 -0.0975"/>
+    </joint>
     <joint name="front_wheel_joint" type="continuous">
+        <axis xyz="0 0 1" />
+        <parent link="bearing_gear"/>
+        <child link="front_wheel"/>
+        <origin xyz="0.0 0.0 -0.0975" rpy="${-pi/2} 0.0 0.0"/>
+        <!--<origin xyz="0.0 0.0 -0.195" rpy="${-pi/2} 0.0 0.0"/--><!---0.195, -0.115-->
+        <!--<origin xyz="0.475 0.0 -0.15" rpy="${-pi/2} 0.0 0.0"/-->
+        <dynamics damping="0.2" />
+    </joint>
+    <!--<joint name="front_wheel_joint" type="continuous">
         <axis xyz="0 0 1" />
         <parent link="chain_frame"/>
@@ -218,4 +256,4 @@
         <origin xyz="-0.1 0.0 -0.085" rpy="${-pi/2} ${pi/2} 0"/>
         <dynamics damping="0.2" />
-    </joint>
+    </joint>-->
 </robot>

File: description/lidar.xacro (robot description, xacro)
@@ -2,7 +2,7 @@
 <robot xmlns:xacro="http://www.ros.org/wiki/xacro" >
     <joint name="laser_joint" type="fixed">
-        <parent link="chassis2"/>
+        <parent link="control_box"/>
         <child link="laser_frame"/>
-        <origin xyz="0.0 0.0 0.195" rpy="0 0 0"/>
+        <origin xyz="0.0 0.0 0.175" rpy="0 0 0"/>
     </joint>
     <link name="laser_frame">

File: description/robot.urdf.xacro (robot description, xacro)
@@ -1,12 +1,15 @@
 <?xml version="1.0"?>
 <robot xmlns:xacro="http://www.ros.org/wiki/xacro"  name="gebot">
-    <xacro:include filename="gebot_core.xacro" />
+    <!--xacro:include filename="gebot_core.xacro" /-->
+    <xacro:include filename="gebot_urdf.xacro" />
     <xacro:include filename="body.xacro" />
     <xacro:include filename="gazebo_material.xacro" />
     <!-- Sensors -->
     <xacro:include filename="lidar.xacro" />
+    <!-- xacro:include filename="camera.xacro" /-->
+    <xacro:include filename="depth_camera.xacro" />
     <!-- Control -->
-    <!-- <xacro:include filename="gazebo_control.xacro" /> -->
-    <!-- <xacro:include filename="ros2_control.xacro" /> -->
+    <!--xacro:include filename="gazebo_control.xacro" /-->
+    <!--xacro:include filename="ros2_control.xacro" /-->
     <xacro:include filename="tricycle_control.xacro" />
     <!-- <xacro:include filename="tricycle_steering_control.xacro" /> -->

File: description/tricycle_control.xacro (robot description, xacro)
@@ -5,6 +5,9 @@
             <plugin>gazebo_ros2_control/GazeboSystem</plugin>
         </hardware>
-        <joint name="front_steering_joint">
+        <!--<joint name="front_steering_joint">-->
+        <joint name="bearing_joint">
             <command_interface name="position"/>
+            <!--command_interface name="angular/position"/-->
+            <!--command_interface name="linear/velocity"/-->
             <state_interface name="position" />
         </joint>
